File: hardware/wearable/sketch.kicad_sch (KiCad schematic)
At the start: 26 parts, among them IC1 LM4041CILPR, U1 INA122P, U2 OPA2350UA, U3 NRF54L15-QFAA-R, Y1 32.768kHz, Y2 32MHz

Commit message: hardware so far
Parts:
- renumbered Rf to Rf2, Rg to Rg1, IC1 to a2
Connections:
- net +3V3: no longer C8.1, U3.10 (VDD), U3.22 (VDD), U3.36 (VDD), U3.47 (VDD), U3.48 (VDD)
- new net: C8.1, U3.10 (VDD), U3.22 (VDD), U3.36 (VDD), U3.47 (VDD), U3.48 (VDD)
Changed lines of the file:
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@@
 		(dnp no)
 		(fields_autoplaced yes)
-		(property "Reference" "IC1"
+		(property "Reference" "a2"
 			(at 31.75 84.5184 0)
 			(effects
@@
 			(project "wearable"
 				(path "/81026750-4f07-481e-af5d-190fa85978a1/f7be8c5b-894c-4046-a913-b3bc16d341b8"
-					(reference "IC1")
+					(reference "a2")
 					(unit 1)
 				)
@@
 		(dnp no)
 		(fields_autoplaced yes)
-		(property "Reference" "Rg"
+		(property "Reference" "Rg1"
 			(at 67.31 27.94 90)
 			(effects
@@
 			(project "wearable"
 				(path "/81026750-4f07-481e-af5d-190fa85978a1/f7be8c5b-894c-4046-a913-b3bc16d341b8"
-					(reference "Rg")
+					(reference "Rg1")
 					(unit 1)
 				)
@@
 		(on_board yes)
 		(dnp no)
-		(property "Reference" "Rf"
+		(property "Reference" "Rf2"
 			(at 125.476 64.516 90)
 			(effects
@@
 			(project "wearable"
 				(path "/81026750-4f07-481e-af5d-190fa85978a1/f7be8c5b-894c-4046-a913-b3bc16d341b8"
-					(reference "Rf")
+					(reference "Rf2")
 					(unit 1)
 				)
@@
 					(unit 1)
 				)
-			)
-		)
-	)
-	(symbol
-		(lib_id "power:+3V3")
-		(at 149.86 119.38 0)
-		(unit 1)
-		(exclude_from_sim no)
-		(in_bom yes)
-		(on_board yes)
-		(dnp no)
-		(fields_autoplaced yes)
-		(property "Reference" "#PWR012"
-			(at 149.86 123.19 0)
-			(effects
-				(font
-					(size 1.27 1.27)
-				)
-				(hide yes)
-			)
-		)
-		(property "Value" "+3V3"
-			(at 149.86 114.3 0)
-			(effects
-				(font
-					(size 1.27 1.27)
-				)
-			)
-		)
-		(property "Footprint" ""
-			(at 149.86 119.38 0)
-			(effects
-				(font
-					(size 1.27 1.27)
-				)
-				(hide yes)
-			)
-		)
-		(property "Datasheet" ""
-			(at 149.86 119.38 0)
-			(effects
-				(font
-					(size 1.27 1.27)
-				)
-				(hide yes)
-			)
-		)
-		(property "Description" "Power symbol creates a global label with name \"+3V3\""
-			(at 149.86 119.38 0)
-			(effects
-				(font
-					(size 1.27 1.27)
-				)
-				(hide yes)
-			)
-		)
-		(pin "1"
-		)
-		(instances
-			(project "wearable"
-				(path "/81026750-4f07-481e-af5d-190fa85978a1/f7be8c5b-894c-4046-a913-b3bc16d341b8"
-					(reference "#PWR012")
-					(unit 1)
-				)
