File: hardware/wearable/wearable.kicad_sch (KiCad schematic)
At the start: 22 parts, among them IC1 LM4041CILPR, U1 INA122P, U2 OPA2350UA

Commit message: updated kicad again..
Parts:
- removed C1, C2: 0.1uF, symbol Device:C_Small
- removed C3, C4, C5, C6: 1uF, symbol Device:C_Small
- removed C7: 1.5uF, symbol Device:C_Small
- removed IC1: LM4041CILPR, ECE445L:ti_LM4041CILPR, symbol ECE445L:LM4041CILPR
- removed R1: 4.7k, symbol Device:R_US
- removed R10, R2: 1k, symbol Device:R_US
- removed R3: 2k, symbol Device:R_US
- removed R4, R9: 1M, symbol Device:R_US
- removed R5, R6: 10k, symbol Device:R_Small_US
- removed R7, R8: 15k, symbol Device:R_US
- removed Rf: 200k, symbol Device:R_US
- removed Rg: 47k, symbol Device:R_US
- removed U1: INA122P, INA122P:DIP794W45P254L959H508Q8, symbol INA122P:INA122P
- removed U2: OPA2350UA, OPA2350UA:SOIC127P599X175-8N, symbol OPA2350UA:OPA2350UA
Other:
- added sheet pcb (pcb.kicad_sch)
- added sheet sketch (sketch.kicad_sch)
- note removed: "HPF fc = ~0.15Hz"
- note removed: "HPF fc = ~15.9Hz"
- note removed: "LPF fc = ~471.5Hz"
- note removed: "Vz = ~1.5V"
- note removed: "gain = 5 + 200k/Rg gain = ~9.25"
