File: hardware/wearable/pcb.kicad_sch (KiCad schematic)
At the start: 1 part, among them U4 INA122U

Commit message: hardware so far
Parts:
- removed U4: INA122U, D8, symbol tat2673custom:INA122U
- added BAT1: 20mm coincell, Sparkfun_LilyPad-Switched-Battery-v1.3:BATTCON_20MM_4LEGS, symbol Sparkfun_LilyPad-Switched-Battery-v1.3-eagle-import:BATTERY20MM_4LEGS
- added C10, C11, C12, C15, C16, C19, C9: 0.1uF, symbol Device:C_Small
- added C13, C14: 0.01uF, symbol Device:C_Small
- added C17: 100nF, symbol Device:C_Small
- added C18, C20, C21, C22: 10uF, symbol Device:C_Small
- added D1, D2, D3, D4: LED, symbol Device:LED
- added IC1: MAX30102EFD+T, MAX30102EFDT, symbol seniorDes:MAX30102EFD+T
- added IC2: INA828IDR, SOIC127P600X175-8N, symbol seniorDes:INA828IDR
- added IC3: LSM6DS3TR-C, LSM6DS3USTR, symbol seniorDes:LSM6DS3TR-C
- added IC4: LM4041CILPR, LM4041CILPR, symbol seniorDes:LM4041CILPR
- added IC5: OPA2350UA, SOIC127P600X175-8N, symbol seniorDes:OPA2350UA
- added IC6: TPS63001DRCT, TPS63001DRCT, symbol seniorDes:TPS63001DRCT
- added J1: Conn_02x05_Odd_Even, symbol Connector_Generic:Conn_02x05_Odd_Even
- added L1: 2.2uH, symbol Device:L_Small
- added R12: 10k, symbol Device:R_Small_US
- added R13: 2.7k, symbol Device:R_Small_US
- added R14: 4.7k, symbol Device:R_Small_US
- added R15, R21: 1k, symbol Device:R_Small_US
- added R16: 5.6k, symbol Device:R_Small_US
- added R17, R18: 100k, symbol Device:R_Small_US
- added R19, R20: 1M, symbol Device:R_Small_US
- added R22, R23: 47k, symbol Device:R_Small_US
- added R24, R25, R26: 100, symbol Device:R_Small_US
- added RN1: 470, YC164JR07470RL, symbol seniorDes:YC164-JR-07470RL
- added Rf1: 200k, symbol Device:R_Small_US
- added SW1: SW_Push, symbol Switch:SW_Push
- added SW2: SW_SPDT, symbol Switch:SW_SPDT
- added U4: BL54L15-453-000xxx, PCM_nordic-lib-kicad-nrf54-modules:BL54Lxx-LGA-39_14x10mm, symbol PCM_nordic-lib-kicad-nrf54-modules:BL54L15-453-000xxx
- added Y4: NX3215SA-32.768K-STD-MUA-8, NX3215SA32768KSTDMUA8, symbol seniorDes:NX3215SA-32.768K-STD-MUA-8
Connections:
- new net: R20.2, R21.1, Rf1.1
- new net: C14.1, IC2.5 (REF), IC4.2, R13.2, R14.1, R17.2, R18.1, R19.2, R21.2
- new net: C12.2, IC5.3 (+IN_A), R19.1
- new net: IC2.1 (RG_1), R16.1
- new net: C10.2, IC2.2 (-IN), R17.1
- new net: C11.2, IC2.3 (+IN), R18.2
- new net: C12.1, IC2.6 (OUT)
- new net: IC2.8 (RG_2), R16.2
- new net: IC5.1 (OUT_A), R22.1, Rf1.2
- new net: C13.2, R22.2, R23.1
- new net: C14.2, IC5.5 (+IN_B), R23.2
- new net: BAT1.POSITIVE@1 (+), BAT1.POSITIVE@2 (+), BAT1.POSITIVE@3 (+), BAT1.POSITIVE@4 (+), SW2.1 (A)
- new net: D3.2 (A), RN1.6
- new net: IC6.2 (L2), L1.2
- new net: IC6.4 (L1), L1.1
- new net: C20.1, IC6.5 (VIN), R26.1, SW2.2 (B)
- new net: C19.1, IC6.6 (EN), IC6.7 (PS/SYNC), IC6.8 (VINA), R26.2
- new net: D1.2 (A), RN1.8
- new net: U4.24 (P1.01), Y4.
- new net: U4.25 (P1.00), Y4.2 (CRYSTAL_2)
- new net: C16.2, R12.2, R25.1, U4.7 (~{RESET})
- new net: D4.2 (A), RN1.5
- new net: IC5.2 (-IN_A), R20.1
- new net: J1.10 (Pin_10), R24.1
- new net: IC4.1, R14.2, R15.1
- new net: D2.2 (A), RN1.7
- new net +3V3: C15.1, C17.1, C18.1, C21.1, C22.1, C9.1, IC2.7 (+VS), IC3.12 (CS), IC3.5 (VDDIO), IC3.8 (VDD), IC5.8 (V+), IC6.1 (VOUT), IC6.10 (FB), J1.1 (Pin_1), R12.1, R13.1, U4.26 (VDD)
- new net Ag+: C11.1
- new net Ag-: C10.1
- new net GND: BAT1.NEGATIVE (-), C15.2, C16.1, C17.2, C18.2, C19.2, C20.2, C21.2, C22.2, C9.2, D1.1 (K), D2.1 (K), D3.1 (K), D4.1 (K), IC1.12 (GND), IC1.4 (PGND), IC2.4 (-VS), IC3.1 (ADO/SA0), IC3.2 (SDX), IC3.3 (SCX), IC3.6 (GND_1), IC3.7 (GND_2), IC4.3, IC5.4 (V-), IC6.11 (PGND_2), IC6.12 (PGND_3), IC6.13 (PGND_4), IC6.14 (PGND_5), IC6.15 (PGND_6), IC6.3 (PGND_1), IC6.9 (GND), J1.3 (Pin_3), J1.5 (Pin_5), R15.2, SW1.2, U4.1 (VSS), U4.16 (VSS), U4.27 (VSS), U4.39 (VSS)
- new net P0.00: U4.17 (P0.00)
- new net P0.01: U4.18 (P0.01)
- new net P0.02: U4.19 (P0.02)
- new net P0.03: IC1.3 (SDA), IC3.14 (SDA), U4.36 (P0.03)
- new net P0.04: U4.31 (P0.04)
- new net P1.02: U4.15 (P1.02)
- new net P1.03: U4.14 (P1.03)
- new net P1.04: C13.1, IC5.6 (-IN_B), IC5.7 (OUT_B), U4.23 (P1.04)
- new net P1.05: IC3.4 (INT1), U4.22 (P1.05)
- new net P1.06: U4.21 (P1.06)
- new net P1.07: U4.20 (P1.07)
- new net P1.08: U4.30 (P1.08)
- new net P1.09: U4.29 (P1.09)
- new net P1.10: U4.28 (P1.10)
- new net P1.11: RN1.1, U4.35 (P1.11)
- new net P1.12: RN1.2, U4.34 (P1.12)
- new net P1.13: RN1.3, U4.33 (P1.13)
- new net P1.14: RN1.4, U4.32 (P1.14)
- new net P2.00: U4.9 (P2.00)
- new net P2.01: U4.10 (P2.01)
- new net P2.02: U4.8 (P2.02)
- new net P2.03: U4.13 (P2.03)
- new net P2.04: U4.11 (P2.04)
- new net P2.05: U4.12 (P2.05)
- new net P2.06: IC1.2 (SCL), IC3.13 (SCL), U4.38 (P2.06)
- new net P2.07: U4.4 (P2.07)
- new net P2.08: U4.3 (P2.08)
- new net P2.09: U4.2 (P2.09)
- new net P2.10: U4.37 (P2.10)
- new net SWDCLK: J1.4 (Pin_4), U4.6 (SWDCLK)
- new net SWDIO: J1.2 (Pin_2), U4.5 (SWDIO)
- new net ~RESET: R24.2, R25.2, SW1.1
- no-connect marks 0 -> 14
Other:
- note added: "HPF fc = ~15.9Hz"
- note added: "Vz = ~1.5V"
- note added: "g = 1 + 50k/Rg"
- note added: "g ≈ 10, Rg = 5.6k"

Commit message: schematic and bom are complete
Parts:
- removed IC3: LSM6DS3TR-C, LSM6DS3USTR, symbol seniorDes:LSM6DS3TR-C
- added C17, C22, C23: 10uF, symbol Device:C_Small
- added C26, C27: 0.1uF, symbol Device:C_Small
- added IC6: TPS62293DRVR, SON65P200X200X80-7N, symbol seniorDes:TPS62293DRVR
- added J2: Conn_01x04_Pin, symbol Connector:Conn_01x04_Pin
- added L2: 2.2uH, symbol Device:L_Small
- added R24: 4.7k, symbol Device:R_Small_US
- added RN2, RN3: 4.7k, C_ARRAY_EXB34V_PAN, symbol seniorDes:EXB34V472JV
- added TP1, TP2, TP3, TP4, TP5, TP6, TP7: TestPoint, symbol Connector:TestPoint
- added U5: LSM6DSOTR, LGA-14L_2P5X3X0P86_STM, symbol seniorDes:LSM6DSOTR
- C11: renamed from C16; value 0.1uF -> 3.9pF
- R12: value 10k -> 4.7k
- renumbered C18 to C10, C10 to C12, C11 to C13, C9 to C14, C12 to C15, C20 to C16, C22 to C18, C21 to C19, C19 to C20, C15 to C21, C13 to C24, C14 to C25, C17 to C9, IC4 to IC1, IC1 to IC3, IC6 to IC4, R13 to R11, R25 to R13, R17 to R16, R18 to R17, R16 to R18, R26 to R20, R20 to R21, R21 to R22, Rf1 to R23, R22 to R25, R23 to R26, R24 to R27, Y4 to Y3
Connections:
- net +3V3: now also IC3.10 (VLED+_2), IC3.9 (VLED+_1), C17.1, C23.2, C26.1, C27.1, IC6.4 (EN), IC6.5 (VIN), R24.1, RN2.1, RN2.2, RN3.3, RN3.4, TP4.1, TP7.1, U5.12 (CS), U5.5 (VDDIO), U5.8 (VDD)
- net GND: now also C17.2, C22.1, C23.1, C26.2, C27.2, IC6.2 (MODE), IC6.6 (GND), U5.1 (SDO/SA0), U5.2 (SDx), U5.3 (SCx), U5.6 (GND), U5.7 (GND)
- net P0.03: now also J2.2 (Pin_2), RN2.3, RN3.1, U5.14 (SDA)
- net P1.04: no longer C24.1, IC5.6 (-IN_B), IC5.7 (OUT_B)
- net P1.05: now also J2.4 (Pin_4), U5.4 (INT1)
- net P1.06: now also C24.1, IC5.6 (-IN_B), IC5.7 (OUT_B), J2.1 (Pin_1)
- net P2.06: now also J2.3 (Pin_3), RN2.4, RN3.2, U5.13 (SCL)
- net ~RESET: now also TP1.1
- net at C25.1, IC1.2, IC2.5 (REF)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: now also TP2.1
- net +1V8: now reaches IC3.11 (VDD)
- net +1V8: now also C22.2, IC6.3 (FB), L2.1, TP5.1, TP6.1
- net at IC3.13 (~{INT}): now also R24.2
- net at BAT1.POSITIVE@1 (+), BAT1.POSITIVE@2 (+), BAT1.POSITIVE@3 (+)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: now also TP3.1
- new net: IC6.1 (SW), L2.2
- no-connect marks 14 -> 15
Other:
- note added: "LPF fc = ~340Hz"
- moved on the sheet: BAT1, C10, C11, C12, C13, C14, C15, C16, C18, C19, C20, C21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

Commit message: working on 3x8cm pcb
Parts:
- added U10, U11, U8, U9: ~, seniorDes:solderPad, symbol seniorDes:solderPad
- added U6, U7: ~, seniorDes:silverContacts, symbol seniorDes:solderPad
- BAT1: footprint Sparkfun_LilyPad-Switched-Battery-v1.3:BATTCON_20MM_4LEGS -> seniorDes:batteryHolder
- C10, C16, C17, C18, C19, C22, C23: footprint (none) -> seniorDes:ceramicCap10uF
- C11: footprint (none) -> seniorDes:ceramicCap3_9pF
- C12, C13, C15: footprint (none) -> seniorDes:C0GCap0_1uF
- C14, C20, C21, C26, C27, C9: footprint (none) -> seniorDes:ceramicCap0_1uF
- C24, C25: footprint (none) -> seniorDes:C0GCap0_01uF
- D1, D2, D3, D4: footprint (none) -> seniorDes:greenLed
- IC1: footprint LM4041CILPR -> seniorDes:lm4041
- IC2: footprint SOIC127P600X175-8N -> seniorDes:ina828
- IC3: footprint MAX30102EFDT -> seniorDes:ppg
- IC4: footprint TPS63001DRCT -> seniorDes:boost3_3v
- IC5: footprint SOIC127P600X175-8N -> seniorDes:opAmp
- IC6: footprint SON65P200X200X80-7N -> seniorDes:buck1_8v
- J1: footprint (none) -> seniorDes:swdConnector
- J2: footprint (none) -> seniorDes:pinHeader1x4
- L1, L2: footprint (none) -> seniorDes:inductor
- R11: footprint (none) -> seniorDes:res2K7
- R12, R14, R24: footprint (none) -> seniorDes:res4K7
- R13, R20, R27: footprint (none) -> seniorDes:res100
- R15, R22: footprint (none) -> seniorDes:res1K
- R16, R17: footprint (none) -> seniorDes:res100K
- R18: footprint (none) -> seniorDes:res5K6
- R19, R21: footprint (none) -> seniorDes:res1M
- R23: footprint (none) -> seniorDes:res200K
- R25, R26: footprint (none) -> seniorDes:red47K
- RN1: footprint YC164JR07470RL -> seniorDes:resArray4
- RN2, RN3: footprint C_ARRAY_EXB34V_PAN -> seniorDes:resArray2
- SW1: footprint (none) -> seniorDes:button
- SW2: footprint (none) -> seniorDes:spdt
- TP1, TP2, TP3, TP4, TP5, TP6, TP7: footprint (none) -> seniorDes:testPoint
- U5: footprint LGA-14L_2P5X3X0P86_STM -> seniorDes:imu
- Y3: footprint NX3215SA32768KSTDMUA8 -> seniorDes:crystal32768
Connections:
- net +3V3: now also RN1.1, RN1.2, RN1.3, RN1.4
- net GND: no longer D1.1 (K), D2.1 (K), D3.1 (K), D4.1 (K)
- net P1.11: now also D4.1 (K); no longer RN1.1
- net P1.12: now also D3.1 (K); no longer RN1.2
- net P1.13: now also D2.1 (K); no longer RN1.3
- net P1.14: now also D1.1 (K); no longer RN1.4
- net ~RESET: no longer TP1.1
- net at U4.24 (P1.01): now also Y3.1; no longer Y3.
- net at C11.2, R12.2, R13.1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: now also TP1.1
- net Ag+: no longer names the net of C13.1
- net Ag+: now also U7.1
- net Ag-: no longer names the net of C12.1
- net Ag-: now also U6.1
- no-connect marks 15 -> 19
Other:
- note added: "Ag+"
- note added: "Ag-"
- note added: "used to solder snaps on (for fabric purposes)"
- moved on the sheet: R13, TP1
